File: getting_started.kicad_sch (KiCad schematic)
At the start: 13 parts, among them J1 Prog connector, J2 Conn_01x03_Pin, U1 STM32F030F4Px, U2 SHT4x

Commit message: Changed debug connector footprint
Parts:
- J1: footprint Connector:Tag-Connect_TC2030-IDC-FP_2x03_P1.27mm_Vertical -> Connector:Tag-Connect_TC2030-IDC-NL_2x03_P1.27mm_Vertical
Changed lines of the file:
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@@
 			)
 		)
-		(property "Footprint" "Connector:Tag-Connect_TC2030-IDC-FP_2x03_P1.27mm_Vertical"
+		(property "Footprint" "Connector:Tag-Connect_TC2030-IDC-NL_2x03_P1.27mm_Vertical"
 			(at 231.14 60.96 0)
 			(effects

Commit message: Updated JST connector
Parts:
- J2: footprint Connector_JST:JST_JWPF_B03B-JWPF-SK-R_1x03_P2.00mm_Vertical -> Connector_JST:JST_XA_B03B-XASK-1-A_1x03_P2.50mm_Vertical
Changed lines of the file:
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@@
 			)
 		)
-		(property "Footprint" "Connector_JST:JST_JWPF_B03B-JWPF-SK-R_1x03_P2.00mm_Vertical"
+		(property "Footprint" "Connector_JST:JST_XA_B03B-XASK-1-A_1x03_P2.50mm_Vertical"
 			(at 50.8 40.64 0)
 			(effects

Commit message: Updated schematic and pcb
Parts:
- removed C2: 100n, Capacitor_SMD:C_0805_2012Metric, symbol Device:C
- removed J1: Prog connector, Connector:Tag-Connect_TC2030-IDC-NL_2x03_P1.27mm_Vertical, symbol Connector:Conn_ARM_SWD_TagConnect_TC2030
- removed J2: Conn_01x03_Pin, Connector_JST:JST_XA_B03B-XASK-1-A_1x03_P2.50mm_Vertical, symbol Connector:Conn_01x03_Pin
- added J1: Conn_01x04_Pin, Connector_JST:JST_XA_B04B-XASK-1-A_1x04_P2.50mm_Vertical, symbol Connector:Conn_01x04_Pin
- added J2: Conn_ARM_JTAG_SWD_10, Connector_PinHeader_1.27mm:PinHeader_2x05_P1.27mm_Vertical, symbol Connector:Conn_ARM_JTAG_SWD_10
- renumbered C3 to C1, C4 to C2, C5 to C3, C6 to C4, C1 to C5, R3 to R2, R4 to R3
Connections:
- net +3.3V: now also J1.2 (Pin_2), J2.1 (VTref)
- net GND: now also U1.10 (PA4), U1.11 (PA5), U1.12 (PA6), U1.13 (PA7), U1.14 (PB1), U1.2 (PF0), U1.3 (PF1), U1.6 (PA0), U1.7 (PA1), J1.1 (Pin_1), J2.3 (GND), J2.5 (GND), J2.6 (SWO/TDO), J2.9 (GNDDetect)
- net SWCLK: now also J2.4 (SWCLK/TCK)
- net SWDIO: now also J2.2 (SWDIO/TMS)
- net IO_RX: now reaches U1.9 (PA3)
- net IO_RX: now also J1.4 (Pin_4)
- net IO renamed IO_TX
- net IO_TX: now also J1.3 (Pin_3)
- net nReset renamed nRESET
- net nRESET: now also J2.10 (~{RESET})
- no-connect marks 11 -> 1
Other:
- note added: "Connector"
- note added: "Debug connector"
- note added: "ERC complicance"
- note added: "MCU and sensor"
- title: Getting started -> Temperature/humidity sensor
- moved on the sheet: C1, C2, C3, C4, C5, R1, R2, R3, U1, U2
